Commit message: urdf_modified

File: urdf_tutorial/urdf_examples/models/unicycle/diff_wheeled_robot.xacro (robot description, xacro)
@@ -79,7 +79,4 @@
         <mass value="${base_mass}" />
         <origin xyz="0 0 0" />
-        <inertia ixx="0.0001" ixy="0.0" ixz="0.0"
-            iyy="0.0001" iyz="0.0"
-            izz="0.0001" />
         <cylinder_inertia  m="${base_mass}" r="${base_radius}" h="${base_height}" />
     </inertial>

Commit message: pan_tilt

File: urdf_tutorial/urdf_examples/models/unicycle/diff_wheeled_robot.xacro (robot description, xacro)
@@ -79,4 +79,7 @@
         <mass value="${base_mass}" />
         <origin xyz="0 0 0" />
+        <inertia ixx="0.0001" ixy="0.0" ixz="0.0"
+            iyy="0.0001" iyz="0.0"
+            izz="0.0001" />
         <cylinder_inertia  m="${base_mass}" r="${base_radius}" h="${base_height}" />
     </inertial>
