Commit message: 2dof

File: ex02/robot_2dof/models/2DoF_arm.xacro (robot description, xacro)
@@ -7,10 +7,29 @@
     <link name = "world"/>
     <joint name="world_joint" type="fixed">
-        <origin xyz="0 0 0" rpy="0 0 0" />
+        <origin xyz="0 0 ${base_height/2}" rpy="0 0 0" />
         <parent link="world"/>
         <child link="chassis"/>
     </joint>
     <!--Chassis-->
-    <xacro:cylinder_link name="chassis" length="${base_height}" radius="${base_width/2}"
-                            z="${base_height/2}" mass="${m1}" colour="Black"/>
+    <xacro:cylinder_link name="chassis" length="${base_height}" radius="${base_width/2}" mass="${m_base}" colour="Black"/>
+    <!--Link 1-->
+    <xacro:cylinder_link name="link1" length="${a1}" radius="${r1}" z="${a1/2}" mass="${m1}" colour="White"/>
+    <!-- Joint 1-->
+    <joint name="joint_1" type="revolute">
+        <origin xyz="0 0 ${base_height/2}" rpy="0 0 0"/>
+        <parent link="chassis"/>
+        <child link="link1"/>
+        <axis xyz="0 1 0"/>
+        <limit effort="${joint_effort}" velocity="${joint_vel}" lower="${-joint_limit}" upper="${joint_limit}"/>
+    </joint>
+    <!--Link 2-->
+    <xacro:cylinder_link name="link2" length="${a2}" radius="${r2}" z="${a2/2}" mass="${m2}" colour="Red"/>
+    <!-- Joint 2-->
+    <joint name="joint_2" type="revolute">
+        <origin xyz="0 0 ${a1}" rpy="0 0 0"/>
+        <parent link="link1"/>
+        <child link="link2"/>
+        <axis xyz="0 1 0"/>
+        <limit effort="${joint_effort}" velocity="${joint_vel}" lower="${-joint_limit}" upper="${joint_limit}"/>
+    </joint>
 </robot>

File: ex02/robot_2dof/models/params_macro.xacro (robot description, xacro)
@@ -21,4 +21,5 @@
     <xacro:property name="r2" value="${props['kinematic_params']['link_radius']}"/>
     <!-- Mass -->
+    <xacro:property name="m_base" value="${props['dynamic_params']['base_mass']}"/> <!--[kg]-->
     <xacro:property name="m1" value="${props['dynamic_params']['m1']}"/>
     <xacro:property name="m2" value="${props['dynamic_params']['m2']}"/>

Commit message: 2dof_dacorreggere

File: ex02/robot_2dof/models/2DoF_arm.xacro (robot description, xacro)
@@ -1,5 +1,5 @@
 <?xml version="1.0"?>
-<robot xmlns:xacro="http://www.ros.org/wiki/xacro" name="ascento">
-    <!-- \\\\\\ Build Ascento Robot \\\\\\ -->
+<robot xmlns:xacro="http://www.ros.org/wiki/xacro" name="2dof_arm">
+    <!-- \\\\\\ Build 2DoF Arm Robot \\\\\\ -->
     <!-- \\\ Include Parameters and Macros \\\ -->
     <xacro:include filename="$(find robot_2dof)/models/params_macro.xacro"/>
@@ -33,3 +33,15 @@
         <limit effort="${joint_effort}" velocity="${joint_vel}" lower="${-joint_limit}" upper="${joint_limit}"/>
     </joint>
+    <!-- \\\ Actuation \\\ -->
+    <!--<xacro:transmission_block joint_name="joint_1" location="1"/>
+    <xacro:transmission_block joint_name="joint_2" location="2"/>-->
+    <!-- \\\\\\ GAZEBO Plugins \\\\\\ -->
+    <!-- ros_control plugin -->
+    <!--<gazebo>
+        <plugin name="gazebo_ros_control" filename="libgazebo_ros_control.so">
+            <robotNamespace>/2dof_arm</robotNamespace>
+            <updateRateHZ>${encoder_freq}</updateRateHZ>
+            <gaussianNoise>${encoder_noise}</gaussianNoise>
+        </plugin>
+    </gazebo>-->
 </robot>

File: ex02/robot_2dof/models/params_macro.xacro (robot description, xacro)
@@ -27,4 +27,7 @@
     <xacro:property name="base_width" value="${props['kinematic_params']['base_width']}"/>
     <xacro:property name="base_height" value="${props['kinematic_params']['base_height']}"/>
+    <!-- \\\ Sensor Data \\\ -->
+    <xacro:property name="encoder_freq" value="${props['encoder']['frequency']}"/>
+    <xacro:property name="encoder_noise" value="${props['encoder']['noise']}"/>
     <!-- \\\\\\ MACRO \\\\\\ -->
     <!-- Inertial Matrix of Cylinder Link -->
@@ -47,5 +50,4 @@
                     <cylinder length="${length}" radius="${radius}"/>
                 </geometry>
-                <material name="${colour}"/>
             </visual>
             <!--Collision: same as Visual-->
@@ -55,5 +57,4 @@
                     <cylinder length="${length}" radius="${radius}"/>
                 </geometry>
-                <material name="${colour}"/>
             </collision>
             <!--Inertial Tensor-->
@@ -68,3 +69,16 @@
         </gazebo>
     </xacro:macro>
+    <!--Transmission Block-->
+    <xacro:macro name="transmission_block" params="joint_name location Type:=Position">
+	  <transmission name="tran_${location}">
+	    <type>transmission_interface/SimpleTransmission</type>
+	    <joint name="${joint_name}">
+	      <hardwareInterface>hardware_interface/${Type}JointInterface</hardwareInterface>
+	    </joint>
+	    <actuator name="motor_${location}">
+	      <hardwareInterface>hardware_interface/${Type}JointInterface</hardwareInterface>
+	      <mechanicalReduction>1</mechanicalReduction>
+	    </actuator>
+	  </transmission>
+    </xacro:macro>
 </robot>

Commit message: correzione2DoF

File: ex02/robot_2dof/models/2DoF_arm.xacro (robot description, xacro)
@@ -7,5 +7,5 @@
     <link name = "world"/>
     <joint name="world_joint" type="fixed">
-        <origin xyz="0 0 ${base_height/2}" rpy="0 0 0" />
+        <origin xyz="0 0 ${base_height}" rpy="0 0 0" />
         <parent link="world"/>
         <child link="chassis"/>
@@ -37,16 +37,15 @@
         <axis xyz="0 1 0"/>
         <limit effort="${joint_effort}" velocity="${joint_vel}" lower="${-joint_limit}" upper="${joint_limit}"/>
+        <dynamics damping="0.0"/>
     </joint>
     <!-- \\\ Actuation \\\ -->
-    <!--<xacro:transmission_block joint_name="joint_1" location="1"/>
-    <xacro:transmission_block joint_name="joint_2" location="2"/>-->
+    <xacro:transmission_block joint_name="joint_1" location="1"/>
+    <xacro:transmission_block joint_name="joint_2" location="2"/>
     <!-- \\\\\\ GAZEBO Plugins \\\\\\ -->
     <!-- ros_control plugin -->
-    <!--<gazebo>
+    <gazebo>
         <plugin name="gazebo_ros_control" filename="libgazebo_ros_control.so">
             <robotNamespace>/2dof_arm</robotNamespace>
-            <updateRateHZ>${encoder_freq}</updateRateHZ>
-            <gaussianNoise>${encoder_noise}</gaussianNoise>
         </plugin>
-    </gazebo>-->
+    </gazebo>
 </robot>

File: ex02/robot_2dof/models/params_macro.xacro (robot description, xacro)
@@ -28,6 +28,4 @@
     <xacro:property name="base_height" value="${props['kinematic_params']['base_height']}"/>
     <!-- \\\ Sensor Data \\\ -->
-    <xacro:property name="encoder_freq" value="${props['encoder']['frequency']}"/>
-    <xacro:property name="encoder_noise" value="${props['encoder']['noise']}"/>
     <!-- \\\\\\ MACRO \\\\\\ -->
     <!-- Inertial Matrix of Cylinder Link -->
@@ -66,4 +64,8 @@
             <static>false</static>
             <turnGravityOff>false</turnGravityOff>
+            <kp>1000000.0</kp>
+            <kd>1.0</kd>
+            <mu1>0.8</mu1>
+            <mu2>0.8</mu2>
             <material>Gazebo/${colour}</material>
         </gazebo>

Commit message: IMU

File: ex02/robot_2dof/models/2DoF_arm.xacro (robot description, xacro)
@@ -49,3 +49,51 @@
         </plugin>
     </gazebo>
+    <!-- IMU Plugins -->
+    <link name="imu_link">
+        <inertial>
+            <mass value="${imu_mass}"/>
+            <inertia ixx="${imu_ixx}" ixy="0.0" ixz="0.0"
+                            iyy="${imu_iyy}" iyz="0.0" izz="${imu_izz}"/>
+            <origin xyz="0 0 0" rpy="0 0 0"/>
+        </inertial>
+        <visual>
+            <origin rpy="0 0 0" xyz="0 0 0"/>
+            <geometry>
+                <box size="${imu_size} ${imu_size} ${imu_size}"/>
+            </geometry>
+        </visual>
+        <collision>
+            <origin rpy="0 0 0" xyz="0 0 0"/>
+            <geometry>
+                <box size="${imu_size} ${imu_size} ${imu_size}"/>
+            </geometry>
+        </collision>
+    </link>
+    <joint name="imu_joint" type="fixed">
+        <axis xyz="1 0 0"/> <!-- 0 1 0 -->
+        <origin xyz="0 0 0"/>
+        <parent link="link2"/>
+        <child link="imu_link"/>
+    </joint>
+    <!-- IMU inherit Sensor Plugin-->
+    <gazebo reference="imu_link">
+        <gravity>true</gravity>
+        <sensor name="imu_sensor" type="imu">
+            <always_on>true</always_on>
+            <update_rate>${imu_freq}</update_rate>
+            <visualize>true</visualize>
+            <topic>__default_topic__</topic>
+            <plugin filename="libgazebo_ros_imu_sensor.so" name="imu_plugin">
+                <topicName>/2dof_arm/imu</topicName>
+                <bodyName>imu_link</bodyName>
+                <updateRateHZ>${imu_freq}</updateRateHZ>
+                <gaussianNoise>${imu_noise}</gaussianNoise>
+                <xyzOffset>0 0 0</xyzOffset>
+                <rpyOffset>0 0 0</rpyOffset>
+                <frameName>imu_link</frameName>
+                <initialOrientationAsReference>false</initialOrientationAsReference>
+            </plugin>
+            <pose>0 0 0 0 0 0</pose>
+        </sensor>
+    </gazebo>
 </robot>

File: ex02/robot_2dof/models/params_macro.xacro (robot description, xacro)
@@ -28,4 +28,11 @@
     <xacro:property name="base_height" value="${props['kinematic_params']['base_height']}"/>
     <!-- \\\ Sensor Data \\\ -->
+    <xacro:property name="imu_mass" value="${props['imu']['mass']}"/>
+    <xacro:property name="imu_ixx" value="${props['imu']['ixx']}"/>
+    <xacro:property name="imu_iyy" value="${props['imu']['iyy']}"/>
+    <xacro:property name="imu_izz" value="${props['imu']['izz']}"/>
+    <xacro:property name="imu_size" value="${props['imu']['size']}"/>
+    <xacro:property name="imu_freq" value="${props['imu']['freq']}"/>
+    <xacro:property name="imu_noise" value="${props['imu']['noise']}"/>
     <!-- \\\\\\ MACRO \\\\\\ -->
     <!-- Inertial Matrix of Cylinder Link -->
